File: CoilDriver.kicad_sch (KiCad schematic)
At the start: 27 parts, among them Q8 IRLML2803, Q9 SiRA99DP, U7 DRV8235RTER

Commit message: Cleaned up silkscreen
Connections:
- net PERI_3V3 is gone; now on net MAIN_3V3: R33.2
Changed lines of the file:
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@@
 			)
 		)
-		(property "Value" "PERI_3V3"
+		(property "Value" "MAIN_3V3"
 			(at 238.76 73.66 0)
 			(effects
