File: ChargeOR.kicad_sch (KiCad schematic)
At the start: 5 parts, among them Q7 SiRA99DP, U6 LTC4412xS6

Commit message: v3.1 Updates
Parts:
- removed Q7: SiRA99DP, Argus-Miscellaneous:PowerPAK SO-8, symbol Argus-IC:Q_PMOS_GDS
- added Q17: SIRA99DP-T1-GE3, Package_SO:PowerPAK_SO-8_Single, symbol Transistor_FET:Si7141DP
- C23: renamed from C10; value 0.1uF -> 100n; MPN (none) -> C307348
- D7: renamed from D2; now left out of the parts list
- F8: renamed from F5; Flight (none) -> 0R
- renumbered U6 to U7
Connections:
- net OUT: now also Q17.1 (S), Q17.2 (S), Q17.3 (S)
- net at C23.1, D7.2 (A), F8.1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: now also Q17.5 (D)
- net at U7.5 (GATE): now also Q17.4 (G)
Other:
- note removed: "#TODO: I think we want to have both of these in parallel"
- company: (none) -> Carnegie Mellon University
- title: (none) -> Argus +Z Solar Panel
- moved on the sheet: D7
Changed lines of the file:
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@@
 (kicad_sch
-	(version 20231120)
+	(version 20250114)
 	(generator "eeschema")
-	(generator_version "8.0")
+	(generator_version "9.0")
 	(paper "A4")
+	(title_block
+		(title "Argus +Z Solar Panel")
+		(date "2025-04-29")
+		(rev "Rev 3.1")
+		(company "Carnegie Mellon University")
+		(comment 1 "N. Khera")
+		(comment 2 "V. Kumar")
+	)
 	(junction
 		(at 146.05 125.73)
@@
 	)
 	(junction
-		(at 158.75 90.17)
+		(at 163.83 90.17)
 		(diameter 0)
 		(color 0 0 0 0)
@@
 	(wire
 		(pts
-			(xy 158.75 72.39) (xy 148.59 72.39)
+			(xy 149.86 74.93) (xy 163.83 74.93)
 		)
 		(stroke
@@
 	(wire
 		(pts
-			(xy 158.75 90.17) (xy 158.75 72.39)
+			(xy 163.83 90.17) (xy 163.83 74.93)
 		)
 		(stroke
@@
 	(wire
 		(pts
+			(xy 151.13 90.17) (xy 163.83 90.17)
+		)
+		(stroke
+			(width 0)
+			(type default)
+		)
+	)
+	(wire
+		(pts
 			(xy 128.27 90.17) (xy 140.97 90.17)
 		)
@@
 	(wire
 		(pts
+			(xy 156.21 110.49) (xy 163.83 110.49)
+		)
+		(stroke
+			(width 0)
+			(type default)
+		)
+	)
+	(wire
+		(pts
 			(xy 146.05 102.87) (xy 146.05 97.79)
 		)
@@
 	(wire
 		(pts
-			(xy 140.97 72.39) (xy 128.27 72.39)
-		)
-		(stroke
-			(width 0)
-			(type default)
-		)
-	)
-	(wire
-		(pts
-			(xy 158.75 90.17) (xy 166.37 90.17)
-		)
-		(stroke
-			(width 0)
-			(type default)
-		)
-	)
-	(wire
-		(pts
-			(xy 151.13 90.17) (xy 158.75 90.17)
+			(xy 142.24 74.93) (xy 128.27 74.93)
+		)
+		(stroke
+			(width 0)
+			(type default)
+		)
+	)
+	(wire
+		(pts
+			(xy 163.83 90.17) (xy 171.45 90.17)
 		)
 		(stroke
@@
 	(wire
 		(pts
-			(xy 128.27 72.39) (xy 128.27 90.17)
-		)
-		(stroke
-			(width 0)
-			(type default)
-		)
-	)
-	(wire
-		(pts
-			(xy 158.75 90.17) (xy 158.75 110.49)
+			(xy 128.27 74.93) (xy 128.27 90.17)
+		)
+		(stroke
+			(width 0)
+			(type default)
+		)
+	)
+	(wire
+		(pts
+			(xy 163.83 90.17) (xy 163.83 110.49)
 		)
 		(stroke
@@
 	(wire
 		(pts
-			(xy 156.21 110.49) (xy 158.75 110.49)
-		)
-		(stroke
-			(width 0)
-			(type default)
-		)
-	)
-	(wire
-		(pts
 			(xy 128.27 110.49) (xy 128.27 115.57)
 		)
@@
 		)
 	)
-	(text "#TODO: I think we want to have both of these in parallel"
-		(exclude_from_sim no)
-		(at 143.764 54.61 0)
+	(hierarchical_label "IN"
+		(shape input)
+		(at 115.57 90.17 180)
 		(effects
 			(font
 				(size 1.27 1.27)
 			)
-		)
-	)
-	(hierarchical_label "IN"
-		(shape input)
-		(at 115.57 90.17 180)
-		(fields_autoplaced yes)
+			(justify right)
+		)
+	)
+	(hierarchical_label "OUT"
+		(shape output)
+		(at 171.45 90.17 0)
 		(effects
 			(font
 				(size 1.27 1.27)
 			)
-			(justify right)
-		)
-	)
-	(hierarchical_label "OUT"
-		(shape output)
-		(at 166.37 90.17 0)
-		(fields_autoplaced yes)
-		(effects
-			(font
-				(size 1.27 1.27)
-			)
 			(justify left)
 		)
@@
 	(symbol
 		(lib_id "Diode:PMEG4005EH")
-		(at 144.78 72.39 180)
+		(at 146.05 74.93 180)
 		(unit 1)
 		(exclude_from_sim no)
-		(in_bom yes)
+		(in_bom no)
 		(on_board yes)
 		(dnp yes)
 		(fields_autoplaced yes)
-		(property "Reference" "D2"
-			(at 145.0975 66.04 0)
+		(property "Reference" "D7"
+			(at 146.3675 68.58 0)
 			(effects
 				(font
@@
 		)
 		(property "Value" "PMEG4005EH"
-			(at 145.0975 68.58 0)
+			(at 146.3675 71.12 0)
 			(effects
 				(font
@@
 		)
 		(property "Footprint" "Diode_SMD:D_SOD-123F"
-			(at 144.78 67.945 0)
+			(at 146.05 70.485 0)
 			(effects
 				(font
@@
 		)
 		(property "Datasheet" "https://assets.nexperia.com/documents/data-sheet/PMEGXX05EH_EJ_SER.pdf"
-			(at 144.78 72.39 0)
+			(at 146.05 74.93 0)
 			(effects
 				(font
@@
 		)
 		(property "Description" "40V, 500mA very low Vf MEGA Schottky barrier rectifier, SOD-123F"
-			(at 144.78 72.39 0)
+			(at 146.05 74.93 0)
 			(effects
 				(font
@@
 			(project "Z+"
 				(path "/977a45af-b6d4-4b54-8e70-e74e2c44e8e7/3495d2a7-7425-4e27-a34a-beb5018fad2a/540f2f39-cb77-4d16-82f8-b8dbe6775262"
-					(reference "D2")
+					(reference "D7")
 					(unit 1)
 				)
@@
 		(on_board yes)
 		(dnp no)
-		(fields_autoplaced yes)
-		(property "Reference" "F5"
+		(property "Reference" "F8"
 			(at 121.92 85.09 0)
 			(effects
@@
 				)
 				(hide yes)
+			)
+		)
+		(property "Flight" "0R"
+			(at 121.92 92.202 0)
+			(effects
+				(font
+					(size 1.27 1.27)
+				)
 			)
 		)
@@
 			(project "Z+"
 				(path "/977a45af-b6d4-4b54-8e70-e74e2c44e8e7/3495d2a7-7425-4e27-a34a-beb5018fad2a/540f2f39-cb77-4d16-82f8-b8dbe6775262"
-					(reference "F5")
+					(reference "F8")
 					(unit 1)
 				)
@@
 		(on_board yes)
 		(dnp no)
-		(property "Reference" "C10"
+		(property "Reference" "C23"
 			(at 126.238 117.094 0)
 			(effects
@@
 			)
 		)
-		(property "Value" "0.1uF"
+		(property "Value" "100n"
 			(at 126.238 119.126 0)
 			(effects
@@
 		)
 		(property "Description" "Unpolarized capacitor, small symbol"
+			(at 128.27 118.11 0)
+			(effects
+				(font
+					(size 1.27 1.27)
+				)
+				(hide yes)
+			)
+		)
+		(property "MPN" "C307348"
 			(at 128.27 118.11 0)
 			(effects
@@
 			(project "Z+"
 				(path "/977a45af-b6d4-4b54-8e70-e74e2c44e8e7/3495d2a7-7425-4e27-a34a-beb5018fad2a/540f2f39-cb77-4d16-82f8-b8dbe6775262"
-					(reference "C10")
+					(reference "C23")
+					(unit 1)
+				)
+			)
+		)
+	)
+	(symbol
+		(lib_id "Transistor_FET:Si7141DP")
+		(at 146.05 92.71 90)
+		(unit 1)
+		(exclude_from_sim no)
+		(in_bom yes)
+		(on_board yes)
+		(dnp no)
+		(property "Reference" "Q17"
+			(at 146.05 84.328 90)
+			(effects
+				(font
+					(size 1.27 1.27)
+				)
+			)
+		)
+		(property "Value" "SIRA99DP-T1-GE3"
+			(at 146.05 86.614 90)
+			(effects
+				(font
+					(size 1.27 1.27)
+				)
+			)
+		)
+		(property "Footprint" "Package_SO:PowerPAK_SO-8_Single"
+			(at 147.955 87.63 0)
+			(effects
+				(font
+					(size 1.27 1.27)
+					(italic yes)
+				)
+				(justify left)
+				(hide yes)
+			)
+		)
+		(property "Datasheet" "https://www.vishay.com/docs/65596/si7141dp.pdf"
+			(at 149.86 87.63 0)
+			(effects
+				(font
+					(size 1.27 1.27)
+				)
+				(justify left)
+				(hide yes)
+			)
+		)
+		(property "Description" "-60A Id, -20V Vds, 1.9 mOhm Ron, PowerPAK-8"
+			(at 146.05 92.71 0)
+			(effects
+				(font
+					(size 1.27 1.27)
+				)
+				(hide yes)
+			)
+		)
+		(property "MPN" "C3289459"
+			(at 146.05 92.71 90)
+			(effects
+				(font
+					(size 1.27 1.27)
+				)
+				(hide yes)
+			)
+		)
+		(pin "5"
+		)
+		(pin "2"
+		)
+		(pin "3"
+		)
+		(pin "4"
+		)
+		(pin "1"
+		)
+		(instances
+			(project "+Z"
+				(path "/977a45af-b6d4-4b54-8e70-e74e2c44e8e7/3495d2a7-7425-4e27-a34a-beb5018fad2a/540f2f39-cb77-4d16-82f8-b8dbe6775262"
+					(reference "Q17")
 					(unit 1)
 				)
@@
 		(dnp no)
 		(fields_autoplaced yes)
-		(property "Reference" "U6"
-			(at 148.2441 100.33 0)
+		(property "Reference" "U7"
+			(at 148.1933 100.33 0)
 			(effects
 				(font
@@
 		)
 		(property "Value" "LTC4412xS6"
-			(at 148.2441 102.87 0)
+			(at 148.1933 102.87 0)
 			(effects
 				(font
@@
 			(project "Z+"
 				(path "/977a45af-b6d4-4b54-8e70-e74e2c44e8e7/3495d2a7-7425-4e27-a34a-beb5018fad2a/540f2f39-cb77-4d16-82f8-b8dbe6775262"
-					(reference "U6")
+					(reference "U7")
 					(unit 1)
 				)
-			)
-		)
-	)
-	(symbol
-		(lib_id "Argus-IC:Q_PMOS_GDS")
-		(at 146.05 92.71 270)
-		(mirror x)
-		(unit 1)
-		(exclude_from_sim no)
-		(in_bom yes)
-		(on_board yes)
-		(dnp no)
-		(property "Reference" "Q7"
-			(at 146.05 83.82 90)
-			(effects
-				(font
-					(size 1.27 1.27)
-				)
-			)
-		)
-		(property "Value" "SiRA99DP"
-			(at 146.05 86.36 90)
-			(effects
-				(font
-					(size 1.27 1.27)
-				)
-			)
-		)
-		(property "Footprint" "Argus-Miscellaneous:PowerPAK SO-8"
-			(at 148.59 87.63 0)
-			(effects
-				(font
-					(size 1.27 1.27)
-				)
-				(hide yes)
-			)
-		)
-		(property "Datasheet" "~"
-			(at 146.05 92.71 0)
-			(effects
-				(font
-					(size 1.27 1.27)
-				)
-				(hide yes)
-			)
-		)
-		(property "Description" "P-MOSFET transistor, gate/drain/source"
-			(at 146.05 92.71 0)
-			(effects
-				(font
-					(size 1.27 1.27)
-				)
-				(hide yes)
-			)
-		)
-		(pin "3"
-		)
-		(pin "2"
-		)
-		(pin "1"
-		)
-		(instances
-			(project "Z+"
-				(path "/977a45af-b6d4-4b54-8e70-e74e2c44e8e7/3495d2a7-7425-4e27-a34a-beb5018fad2a/540f2f39-cb77-4d16-82f8-b8dbe6775262"
-					(reference "Q7")
-					(unit 1)
-				)
