File: I2CSingleProtection.kicad_sch (KiCad schematic)
At the start: 9 parts, among them Q14 NX3008NBKS, Q15 MBT2222ADW1T1

Commit message: v3.1 Updates
Parts:
- C5: renamed from C27; value 10nF -> 10n; symbol Device:C -> Device:C_Small; MPN (none) -> C161232
- Q2: renamed from Q14; MPN (none) -> C3280240; Manufacturer_Name Nexperia USA Inc. -> (none); Manufacturer_Part_Number NX3008NBKS -> (none)
- R10: renamed from R64; value DNI (0R) -> 0R; now not fitted; now left out of the parts list
- R5: renamed from R65; value 10K -> 10k; MPN (none) -> C2479067
- R6: renamed from R66; value 10K -> 10k; MPN (none) -> C2479067
- R7: renamed from R62; MPN (none) -> C844802
- R8: renamed from R63; value 100K -> 100k; MPN (none) -> C237792
- R9: renamed from R67; value 200K -> 200k; MPN (none) -> C118142
- renumbered Q15 to Q1
Other:
- company: (none) -> Carnegie Mellon University
- title: (none) -> Argus +Z Solar Panel
