File: MPPT.kicad_sch (KiCad schematic)
At the start: 15 parts, among them U9 LTC3130

Commit message: v3.1 Updates
Parts:
- C14: renamed from C18; value 47uF -> 47u
- C15: renamed from C19; value 10uF -> 10u; MPN (none) -> C126617; Mfr. # C1608X7S1A475K080AC -> (none); Order https://www.digikey.com/product-detail/en/tdk-corporation/C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 -> (none); Voltage 10V -> (none)
- C16: renamed from C20; value 1uF -> 1u; MPN (none) -> C2214844; Mfr. # C1608X7S1A475K080AC -> (none); Order https://www.digikey.com/product-detail/en/tdk-corporation/C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 -> (none); Voltage 10V -> (none)
- C17: renamed from C21; value 1uF -> 1u; MPN (none) -> C2214844; Mfr. # CL10B105KP8NFNC -> (none); Order https://www.digikey.com/product-detail/en/samsung-electro-m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 -> (none); Voltage 10V -> (none)
- C18: renamed from C22; value 22nF -> 22n
- C19: renamed from C23; value 22nF -> 22n
- C20: renamed from C25; value 1uF -> 1u; MPN (none) -> C2214844; Mfr. # GRM32EC81C476KE15L -> (none); Order https://www.digikey.com/product-detail/en/murata-electronic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 -> (none); Voltage 16V -> (none)
- C21: renamed from C26; value 47uF -> 47u
- C22: renamed from C24; value 4.7uF -> 4u7; MPN (none) -> C437575; Mfr. # C1608X7S1A475K080AC -> (none); Order https://www.digikey.com/product-detail/en/tdk-corporation/C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 -> (none); Voltage 10V -> (none)
- L1: value 6.8uH -> 6.8u
- R64: renamed from R58; value 0R (DNI) -> 0R; DNI (none) -> DNI; Mfr. # RK73Z1JTTDr -> (none); Order https://www.digikey.com/product-detail/en/koa-speer-electro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 -> (none); now not fitted; now left out of the parts list
- R65: renamed from R59; MPN (none) -> C844915; Mfr. # RK73Z1JTTDr -> (none); Order https://www.digikey.com/product-detail/en/koa-speer-electro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 -> (none)
- R66: renamed from R60; MPN (none) -> C844915; Mfr. # RK73Z1JTTDr -> (none); Order https://www.digikey.com/product-detail/en/koa-speer-electro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 -> (none)
- R67: renamed from R61; MPN (none) -> C844915; Mfr. # RK73Z1JTTDr -> (none); Order https://www.digikey.com/product-detail/en/koa-speer-electro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 -> (none)
- U6: renamed from U9; value LTC3130 -> LTC3130IUDC; MPN (none) -> C684244
Other:
- company: (none) -> Carnegie Mellon University
- title: (none) -> Argus +Z Solar Panel
- moved on the sheet: C17, C18, C19, C22, L1
