File: MPPT.kicad_sch (KiCad schematic)
At the start: 15 parts, among them U6 LTC3130IUDC

Commit message: Re-Exported BOM
Parts:
- C18, C19: MPN (none) -> C161234; Mfr. # GCM188R72A223KA37D -> (none); Order https://www.digikey.com/product-detail/en/murata-electronic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 -> (none); Voltage 100V -> (none)
Changed lines of the file:
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@@
 			)
 		)
-		(property "Mfr. #" "GCM188R72A223KA37D"
+		(property "MPN" "C161234"
 			(at 157.48 66.04 90)
-			(effects
-				(font
-					(size 1.27 1.27)
-				)
-				(hide yes)
-			)
-		)
-		(property "Order" "https://www.digikey.com/product-detail/en/murata-electronics/GCM188R72A223KA37D/490-4782-1-ND/1641701"
-			(at 157.48 66.04 90)
-			(effects
-				(font
-					(size 1.27 1.27)
-				)
-				(hide yes)
-			)
-		)
-		(property "Voltage" "100V"
-			(at 157.48 69.215 90)
 			(effects
 				(font
@@
 			)
 		)
-		(property "Mfr. #" "GCM188R72A223KA37D"
+		(property "MPN" "C161234"
 			(at 180.34 66.04 90)
 			(effects
 				(font
-					(size 1.27 1.27)
-				)
-				(hide yes)
-			)
-		)
-		(property "Order" "https://www.digikey.com/product-detail/en/murata-electronics/GCM188R72A223KA37D/490-4782-1-ND/1641701"
-			(at 180.34 66.04 90)
-			(effects
-				(font
-					(size 1.27 1.27)
-				)
-				(hide yes)
-			)
-		)
-		(property "Voltage" "100V"
-			(at 180.34 69.215 90)
-			(effects
-				(font
