File: SolarCharger.kicad_sch (KiCad schematic)
At the start: 30 parts, among them U8 ADM1176-1ARMZ-R7

Commit message: v3.1 Updates
Parts:
- removed R109, R57: 0R, Resistor_SMD:R_0603_1608Metric, symbol Device:R_Small
- C13: renamed from C17; value 3.3nF -> 3n3; MPN (none) -> C3877267
- D1: renamed from D5; value DFLS130L-7 -> DFLS130LQ-7
- D2: renamed from D6; value DFLS130L-7 -> DFLS130LQ-7
- D3: renamed from D7; value DFLS130L-7 -> DFLS130LQ-7
- D4: renamed from D8; value DFLS130L-7 -> DFLS130LQ-7
- D5: renamed from D9; value DFLS130L-7 -> DFLS130LQ-7
- D6: renamed from D10; value DFLS130L-7 -> DFLS130LQ-7
- F5: renamed from F7; value 100mA -> 500mA; Flight (none) -> 0R
- R53: renamed from R55; value ?R -> 10m; MPN (none) -> C840621
- R54: renamed from R56; value 1K -> 1k; MPN (none) -> C2484712
- R55: renamed from R108; DNI (none) -> DNI; now not fitted; now left out of the parts list
- R56: renamed from R110; MPN (none) -> C844915
- R61: renamed from R52; value 100K -> 100k; MPN (none) -> C237792
- R63: renamed from R54; value 200K -> 200k; MPN (none) -> C118142
- SC1, SC2, SC3, SC4, SC5, SC6: value SM141K06TF -> SM141K06TF/S; footprint Argus-Miscellaneous:SM141K06TF -> Argus-Miscellaneous:SM141K06TF_S
- renumbered F8 to F6, F9 to F7, R49 to R57, R50 to R58, R48 to R59, R51 to R60, R53 to R62, U8 to U5
Connections:
- net MPPT/VIN is gone; now on net VSOLAR: F5.1, R57.1, R59.1
- net VSOLAR: no longer D6.1 (K), F5.2, SC6.1 (+)
- net at F7.1, U5.2 (SENSE): now also R54.2; no longer R54.1
- net at U5.3 (ON): now also R54.1; no longer R54.2
- net A0_S renamed A0
- net A1_S renamed A1
- net PGOOD3 renamed PGOOD
- new net: D6.1 (K), F5.2, SC6.1 (+)
Other:
- sheet Charge OR-ing2 renamed Charge OR-ing
- sheet I2C Single Protection4 renamed I2C Single Protection8
- sheet I2C Single Protection5 renamed I2C Single Protection9
- sheet MPPT2 renamed MPPT
- note added: "#TODO: Check Resistor Values"
- note added: "#TODO: Spec Fuses"
- note added: "I2C ADDR R55, R56 +Z: DNP, 0R: 0x42 Translated: 0x62"
- note added: "Rsense"
- note removed: "#TODO: Recalculate values for 6S solar panels"
- note removed: "I2C ADDR 0x94 Install R66: 0x90"
- company: (none) -> Carnegie Mellon University
- title: (none) -> Argus +Z Solar Panel
- moved on the sheet: C13, D1, D2, D3, D4, D5, D6, F5, F6, F7, R53, R54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
