File: SunPyramid.kicad_sch (KiCad schematic)
At the start: 16 parts, among them U2 SunSensor, U3 SunSensor, U4 SunSensor, U5 SunSensor

Commit message: v3.1 Updates
Parts:
- C1: renamed from C8; value 100nF -> 100n; MPN (none) -> C307348
- C2: renamed from C5; value 100nF -> 100n; MPN (none) -> C307348
- C3: renamed from C6; value 100nF -> 100n; MPN (none) -> C307348
- C4: renamed from C7; value 100nF -> 100n; MPN (none) -> C307348
- F1, F2, F3, F4: value Fuse_Small -> 100mA
- R1: renamed from R104; MPN (none) -> C844915
- R2: renamed from R105; MPN (none) -> C844915
- R3: renamed from R106; MPN (none) -> C844915
- R4: renamed from R107; MPN (none) -> C844915
- renumbered U2 to U1, U3 to U2, U4 to U3, U5 to U4
Connections:
- net PERI_3V3 renamed 3V3_P
Other:
- sheet I2C Single Protection10 renamed I2C Single Protection5
- sheet I2C Single Protection9 renamed I2C Single Protection4
- removed sheet I2C Single Protection11
- removed sheet I2C Single Protection12
- removed sheet I2C Single Protection8
- added sheet I2C Single Protection (I2CSingleProtection.kicad_sch)
- added sheet I2C Single Protection1 (I2CSingleProtection.kicad_sch)
- added sheet I2C Single Protection2 (I2CSingleProtection.kicad_sch)
- note added: "+X SUN SENSOR I2C ADDR 0x45 Translated: 0x65"
- note added: "+Y SUN SENSOR I2C ADDR 0x44 Translated: 0x64"
- note added: "-X SUN SENSOR I2C ADDR 0x47 Translated: 0x67"
- note added: "-Y SUN SENSOR I2C ADDR 0x46 Translated: 0x66"
- company: (none) -> Carnegie Mellon University
- title: (none) -> Argus +Z Solar Panel
- moved on the sheet: C1, C2, C3, C4, F1, F2, F3, F4, R1, R2, R3, R4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
