File: I2C_Translator.kicad_sch (KiCad schematic)
At the start: 14 parts, among them U11 LTC4316xDD

Commit message: v3.1 Updates
Parts:
- C33: renamed from C35; value 0.1uF -> 100n; symbol SolarPanels:C_Small -> Device:C_Small; MPN (none) -> C307348
- R107: renamed from R121; value 10K -> 10k; symbol SolarPanels:R_Small -> Device:R_Small; MPN (none) -> C2479067
- R108: renamed from R122; value 10K -> 10k; symbol SolarPanels:R_Small -> Device:R_Small; MPN (none) -> C2479067
- R109: renamed from R123; value 10K -> 10k; symbol SolarPanels:R_Small -> Device:R_Small; MPN (none) -> C2479067
- R110: renamed from R117; value ? -> 0R; symbol SolarPanels:R_Small -> Device:R_Small; DNI (none) -> DNI; now not fitted; now left out of the parts list
- R111: renamed from R118; value ? -> 0R; symbol SolarPanels:R_Small -> Device:R_Small; MPN (none) -> C844915
- R112: renamed from R119; value ? -> 976k; symbol SolarPanels:R_Small -> Device:R_Small
- R113: renamed from R120; value ? -> 102k; symbol SolarPanels:R_Small -> Device:R_Small
- R114: renamed from R126; value 0R (DNI) -> 0R; symbol SolarPanels:R_Small -> Device:R_Small; DNI (none) -> DNI; now not fitted; now left out of the parts list
- R115: renamed from R124; symbol SolarPanels:R_Small -> Device:R_Small; MPN (none) -> C844915
- R116: renamed from R127; value 0R (DNI) -> 0R; symbol SolarPanels:R_Small -> Device:R_Small; DNI (none) -> DNI; now not fitted; now left out of the parts list
- R117: renamed from R125; symbol SolarPanels:R_Small -> Device:R_Small; MPN (none) -> C844915
- U10: renamed from U11; value LTC4316xDD -> LTC4316IDD; MPN (none) -> C688147
Connections:
- net SCL_MB is gone; now on net SCL: R114.2, U10.10 (SCLIN)
- net SDA_MB is gone; now on net SDA: R116.2, U10.7 (SDAIN)
- net SCL: no longer R114.1, R115.1
- net SDA: no longer R116.1, R117.1
- net PERI_3V3 renamed 3V3_P
- new net SCL_LS: R114.1, R115.1
- new net SDA_LS: R116.1, R117.1
Other:
- note added: "Translation Byte: 0x20 #TODO: Test Resistor Values"
- company: (none) -> Carnegie Mellon University
- title: (none) -> Argus +Z Solar Panel
- moved on the sheet: C33, F10, R107, R108, R109, R111, R112, R113, R115, R117, U10
