File: Interfaces.kicad_sch (KiCad schematic)
At the start: 0 parts

Commit message: v3.1 Updates
Parts:
- added C32: 100n, Capacitor_SMD:C_0603_1608Metric, symbol Device:C_Small
- added J1: 522711069, Argus-Connectors:CON_522711069_MOL, symbol Connector_Generic_MountingPin:Conn_01x10_MountingPin
- added U9: D5V0P4UR6SO, Package_TO_SOT_SMD:SOT-23-6, symbol Power_Protection:SRV05-4
Connections:
- new net 3V3_P: C32.1, J1.4 (Pin_4), J1.5 (Pin_5), U9.5 (VP)
- new net COIL_DRIVER_EN: J1.3 (Pin_3)
- new net GND: C32.2, J1.6 (Pin_6), J1.7 (Pin_7), J1.MP (MountPin), U9.2 (VN)
- new net SCL: J1.1 (Pin_1), U9.1 (IO1)
- new net SDA: J1.2 (Pin_2), U9.3 (IO2)
- new net VBATT: J1.10 (Pin_10), J1.8 (Pin_8), J1.9 (Pin_9)
- no-connect marks 0 -> 2
Other:
- removed sheet Mainboard FPC
- removed sheet RBF
- removed sheet USB-C
- company: (none) -> Carnegie Mellon University
- title: (none) -> Argus +Z Solar Panel
