File: LightSensorBreakout/LightSensorBreakout.kicad_pcb (KiCad board)
At the start: 2 copper layers, 22 x 4 mm, 6 parts, among them U1 OPT4003DNPRQ1

Commit message: V4 Updates
Routing:
- net /SDA: track 13.1 -> 13.7 mm
Other:
- board text added: "ARGUS CUBESAT"
